File: public/examples/pcbplanner-example-6layer.kicad_pcb (KiCad board)
At the start: 6 copper layers, 80 x 60 mm, 4 parts, among them J1 +5V in, U1 AMS1117-3.3, U2 MCU

Commit message: Complete KiCad analysis workflows, project reports and teaching board
Parts:
- added C2: Input bulk (demo), Capacitor_SMD:C_0603_1608Metric, F.Cu at (132.0, 152.0)
- added C3: Output bulk (demo), Capacitor_SMD:C_0603_1608Metric, F.Cu at (146.0, 153.7)
- added J2: Routing coupon, PCBPlanner:Routing_Coupon_Pads, F.Cu at (130.0, 118.0)
- added J3: Routing coupon, PCBPlanner:Routing_Coupon_Pads, F.Cu at (175.0, 118.0)
- added J4: Routing coupon, PCBPlanner:Routing_Coupon_Pads, F.Cu at (130.0, 108.0)
- added J5: Routing coupon, PCBPlanner:Routing_Coupon_Pads, F.Cu at (130.0, 124.0)
- added J6: Routing coupon, PCBPlanner:Routing_Coupon_Pads, F.Cu at (161.0, 138.0)
- added J8: 48V clearance coupon, Connector_PinHeader_2.54mm:PinHeader_1x02_P2.54mm_Vertical, F.Cu at (108.0, 113.0)
- added R1: 10k (clearance coupon), Resistor_SMD:R_0805_2012Metric, F.Cu at (119.0, 125.0)
- added TP1: CLK, PCBPlanner:TestPad, F.Cu at (130.0, 150.0)
- added TP2: SDA, PCBPlanner:TestPad, F.Cu at (110.0, 140.0)
- added TP3: SDA, PCBPlanner:TestPad, F.Cu at (110.0, 150.0)
- added TP4: CLK, PCBPlanner:TestPad, F.Cu at (110.0, 145.0)
- U1: value AMS1117-3.3 -> 3.3V regulator (demo)
- U2: value MCU -> 3.3V load (demo); footprint Package_DFN_QFN:QFN-16-1EP_4x4mm_P0.65mm -> PCBPlanner:Demo_Load_ExposedPad
Routing:
- net /SDA: track 110.0 -> 134.2 mm, vias 0 -> 3
- net +48V: track 0.00 -> 23.3 mm
- net GND: track 47.7 -> 56.7 mm, vias 7 -> 11
- net /CLK: track 100.0 -> 105.0 mm, vias 0 -> 2
- net +5V: track 18.7 -> 20.5 mm, vias 1 -> 2
- net +3V3: track 36.6 -> 37.7 mm, vias 0 -> 3
Other:
- board text added: "0.35 mm GAP"
- board text added: "3.3 V LOAD"
- board text added: "3.3 V REGULATOR"
- board text added: "48 V / CLEARANCE"
- board text added: "5 V IN"
- board text added: "CLOCK / ROUTING COUPONS"
- board text added: "HDMI / BEND SKEW"
- board text added: "INTENTIONAL FINDINGS"
- board text added: "NOT FOR FABRICATION"
- board text added: "PCB PLANNER / 6-LAYER LAB"
- board text added: "PCIe / MATCHED PAIR"
- board text added: "TEACHING BOARD"
- board text added: "USB / LAYER CHANGE"
